Commit message: hw working

File: src/servera_description/hw_urdf/hw_lidar.xacro (robot description, xacro)
@@ -4,5 +4,5 @@
     <link name="${frame_id}">
       <visual>
-        <origin xyz="0 0 -0.025" rpy="0 0 0"/>
+        <origin xyz="0 0 0.025" rpy="0 0 0"/>
         <geometry>
           <cylinder radius="0.0375" length="0.05"/>
@@ -12,20 +12,4 @@
         </material>
       </visual>
-      <collision>
-        <origin xyz="0 0 -0.025" rpy="0 0 0"/>
-        <geometry>
-          <cylinder radius="0.0375" length="0.05"/>
-        </geometry>
-      </collision>
-      <inertial>
-        <origin xyz="0 0 0" rpy="0 0 0"/>
-        <mass value="0.1"/>
-        <inertia ixx="${(1/12) * 0.1 * (3 * 0.0375 * 0.0375 + 0.05 * 0.05)}"
-                 ixy="0"
-                 ixz="0"
-                 iyy="${(1/12) * 0.1 * (3 * 0.0375 * 0.0375 + 0.05 * 0.05)}"
-                 iyz="0"
-                 izz="${(1/2) * 0.1 * (0.0375 * 0.0375)}" />
-      </inertial>
     </link>
     <joint name="${frame_id}_to_base_link" type="fixed">

File: src/servera_description/hw_urdf/servera_hw.urdf.xacro (robot description, xacro)
@@ -38,5 +38,5 @@
     <xacro:lidar
         frame_id="lidar_link" >
-        <origin xyz="0.0 0.0 ${base_height}" rpy="0 0 0"/>
+        <origin xyz="0.0 0.0 ${base_height-wheel_radius}" rpy="0 0 3.14"/>
     </xacro:lidar>
     <xacro:caster_wheel

File: src/servera_description/hw_urdf/servera_properties.xacro (robot description, xacro)
@@ -1,14 +1,14 @@
 <?xml version="1.0"?>
 <robot xmlns:xacro="http://ros.org/wiki/xacro">
-  <xacro:property name="base_length" value="0.5" />
-  <xacro:property name="base_width" value="0.3" />
-  <xacro:property name="base_height" value="0.2" />
-  <xacro:property name="base_mass" value="1" />
-  <xacro:property name="wheel_radius" value="0.045" />
-  <xacro:property name="wheel_width" value="0.025" />
-  <xacro:property name="wheel_pos_x" value="0.03" />
-  <xacro:property name="wheel_pos_y" value="0.165" />
-  <xacro:property name="wheel_pos_z" value="-0.03" />
-  <xacro:property name="wheel_mass" value=".1" />
+  <xacro:property name="base_length" value="1.2" />
+  <xacro:property name="base_width" value="0.590" />
+  <xacro:property name="base_height" value="0.625" />
+  <xacro:property name="base_mass" value="50" />
+  <xacro:property name="wheel_radius" value="0.1" />
+  <xacro:property name="wheel_width" value="0.05" />
+  <xacro:property name="wheel_pos_x" value="0.05" />
+  <xacro:property name="wheel_pos_y" value="0.325" />
+  <xacro:property name="wheel_pos_z" value="-0.1" />
+  <xacro:property name="wheel_mass" value=".3" />
   <xacro:property name="wheel_torque" value="20" />
   <xacro:property name="front_caster_wheel" value="true" />
