Commit message: feb update

File: src/servera_control/urdf/gz_lidar.xacro (robot description, xacro)
@@ -52,6 +52,6 @@
         <!-- <frame_id>${frame_id}</frame_id> -->
         <update_rate>${update_rate}</update_rate>
-        <always_on>1</always_on>
-        <visualize>1</visualize>
+        <always_on>true</always_on>
+        <visualize>true</visualize>
         <lidar>
           <scan>
@@ -62,4 +62,10 @@
               <max_angle>${max_angle}</max_angle>
             </horizontal>
+            <vertical>
+              <samples>1</samples>
+              <resolution>1</resolution>
+              <min_angle>0.0</min_angle>
+              <max_angle>0.0</max_angle>
+            </vertical>
           </scan>
           <range>

File: src/servera_control/urdf/servera.urdf.xacro (robot description, xacro)
@@ -44,5 +44,5 @@
         frame_id="lidar_link"
         topic_name="scan">  <!-- Do not use "/" for topic names, ie "/scan"; instead use "scan"-->
-        <origin xyz="0.0 0.0 ${base_height}" rpy="0 0 0"/>
+        <origin xyz="0.0 0.0 ${base_height-wheel_radius}" rpy="0 0 0"/>
     </xacro:lidar>
     <xacro:caster_wheel

File: src/servera_control/urdf/servera_properties.xacro (robot description, xacro)
@@ -1,14 +1,14 @@
 <?xml version="1.0"?>
 <robot xmlns:xacro="http://ros.org/wiki/xacro">
-  <xacro:property name="base_length" value="0.5" />
-  <xacro:property name="base_width" value="0.3" />
-  <xacro:property name="base_height" value="0.2" />
-  <xacro:property name="base_mass" value="1" />
-  <xacro:property name="wheel_radius" value="0.045" />
-  <xacro:property name="wheel_width" value="0.025" />
-  <xacro:property name="wheel_pos_x" value="0.03" />
-  <xacro:property name="wheel_pos_y" value="0.165" />
-  <xacro:property name="wheel_pos_z" value="-0.03" />
-  <xacro:property name="wheel_mass" value=".1" />
+  <xacro:property name="base_length" value="1.2" />
+  <xacro:property name="base_width" value="0.6" />
+  <xacro:property name="base_height" value="0.625" />
+  <xacro:property name="base_mass" value="50" />
+  <xacro:property name="wheel_radius" value="0.1" />
+  <xacro:property name="wheel_width" value="0.05" />
+  <xacro:property name="wheel_pos_x" value="0.05" />
+  <xacro:property name="wheel_pos_y" value="0.325" />
+  <xacro:property name="wheel_pos_z" value="-0.1" />
+  <xacro:property name="wheel_mass" value=".3" />
   <xacro:property name="wheel_torque" value="20" />
   <xacro:property name="front_caster_wheel" value="true" />
