Commit message: march update

File: src/servera_description/urdf/gz_lidar.xacro (robot description, xacro)
@@ -4,5 +4,5 @@
     <link name="${frame_id}">
       <visual>
-        <origin xyz="0 0 -0.025" rpy="0 0 0"/>
+        <origin xyz="0 0 0" rpy="0 0 0"/>
         <geometry>
           <cylinder radius="0.0375" length="0.05"/>

File: src/servera_description/urdf/servera.urdf.xacro (robot description, xacro)
@@ -6,4 +6,5 @@
     <xacro:include filename="$(find servera_description)/urdf/material.xacro"/>  <!-- All the meterial list | consemtics -->
     <xacro:include filename="$(find servera_description)/urdf/gz_plugins.xacro"/>  <!-- gz tags | gz integrartion -->
+    <xacro:include filename="$(find servera_description)/urdf/orbbec_gem336l.xacro"/>
     <xacro:base
         length="${base_length}"
@@ -44,5 +45,5 @@
         frame_id="lidar_link"
         topic_name="/scan">
-        <origin xyz="0.0 0.0 ${base_height}" rpy="0 0 0"/>
+        <origin xyz="0.0 0.0 ${base_height-wheel_radius+0.025}" rpy="0 0 0"/>
     </xacro:lidar>
     <xacro:caster_wheel
@@ -62,3 +63,7 @@
       wheel_pos_z="${wheel_pos_z}"
     />
+    <xacro:gemini_336l
+    parent="base_link"
+    xyz="0.62 0.035 0.3"
+    rpy="0 0 0"/>
 </robot>
